File: Scout_Board.kicad_pcb (KiCad board)
At the start: 2 copper layers, 102.5 x 80 mm, 56 parts, among them J1 Conn_01x01_Pin, J2 Conn_01x04_Pin, J3 RAPC722X, J4 5V, J5 GND, Q1 BSS138, Q2 BSS138, U1 DRV8871DDA, U2 ESP32-S3-DEVKITC-1U-N8R2, U3 LM2576HVS-5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

Commit message: a
Routing:
- net +12V: track 0.00 -> 60.2 mm
Changed lines of the file:
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@@
   (gr_circle locked (center 234.93 92.456) (end 236.43 92.456)
     (stroke (width 0.1) (type default)) (fill none) (layer "Edge.Cuts"))
+  (segment (start 205.232 107.188) (end 203.2 109.22) (width 0.25) (layer "F.Cu") (net 1))
+  (segment (start 226.568 98.706) (end 226.568 100.838) (width 0.25) (layer "F.Cu") (net 1))
+  (segment (start 216.98 133.096) (end 210.884 127) (width 0.25) (layer "F.Cu") (net 1))
+  (segment (start 225.996 101.282) (end 212.598 101.282) (width 0.25) (layer "F.Cu") (net 1))
+  (segment (start 224.662 133.096) (end 216.98 133.096) (width 0.25) (layer "F.Cu") (net 1))
+  (segment (start 212.598 101.282) (end 210.502 103.378) (width 0.25) (layer "F.Cu") (net 1))
+  (segment (start 196.454 109.22) (end 194.974 107.74) (width 0.25) (layer "F.Cu") (net 1))
+  (segment (start 226.216 134.65) (end 224.662 133.096) (width 0.25) (layer "F.Cu") (net 1))
+  (segment (start 210.502 103.378) (end 206.502 103.378) (width 0.25) (layer "F.Cu") (net 1))
+  (segment (start 194.974 107.74) (end 194.974 105.44) (width 0.25) (layer "F.Cu") (net 1))
+  (segment (start 226.06 101.346) (end 225.996 101.282) (width 0.25) (layer "F.Cu") (net 1))
+  (segment (start 206.502 103.378) (end 205.232 104.648) (width 0.25) (layer "F.Cu") (net 1))
+  (segment (start 205.232 104.648) (end 205.232 107.188) (width 0.25) (layer "F.Cu") (net 1))
+  (segment (start 203.2 109.22) (end 196.454 109.22) (width 0.25) (layer "F.Cu") (net 1))
+  (segment (start 226.568 100.838) (end 226.06 101.346) (width 0.25) (layer "F.Cu") (net 1))
   (zone (net 2) (net_name "GND") (layer "F.Cu") (hatch edge 0.5)
     (connect_pads (clearance 0.5))

Commit message: Pcb - no errors
Parts:
- added J4: Screw_Terminal_01x02, TerminalBlock_MetzConnect:TerminalBlock_MetzConnect_Type011_RT05502HBWC_1x02_P5.00mm_Horizontal, F.Cu at (180.9, 97.3)
- moved C2 34.1 mm to (193.8, 126.2)
- moved J1 20.4 mm to (172.5, 148.8)
- moved D2 18.6 mm to (229.9, 138.9), turned to 0 degrees
- moved C1 18.5 mm to (173.2, 99.3), turned to -90 degrees
- moved R1 10.7 mm to (169.4, 99.3), turned to -90 degrees
- moved D1 6.93 mm to (205.5, 114.8), turned to -90 degrees
- moved L1 1.55 mm to (214.1, 112.0)
- moved C5 1.27 mm to (230.4, 146.1)
- moved R9 0.25 mm to (187.5, 122.8), turned to 90 degrees
- turned U2 to 180 degrees
- renumbered J4 to J5, J5 to J6
Connections:
- C3 pad 1: +5V -> +5VA
- Conn5 pad 1: (no net) -> +12V
- Conn5 pad 2: (no net) -> Net-(Conn5-Pin_2)
- L1 pad 2: +5V -> +5VA
- U3 pad 4: +5V -> +5VA
Routing:
- net +5V: track 0.00 -> 169.7 mm
- net Sw1: track 0.00 -> 138.5 mm, vias 0 -> 2
- net Button5: track 0.00 -> 111.4 mm, vias 0 -> 1
- net Button3: track 0.00 -> 109.2 mm, vias 0 -> 2
- net CaptureButton: track 0.00 -> 107.3 mm, vias 0 -> 2
- net Button4: track 0.00 -> 106.8 mm, vias 0 -> 2
- net +12V: track 60.2 -> 160.4 mm
- net Button6: track 0.00 -> 93.7 mm, vias 0 -> 1
- net FlipButton: track 0.00 -> 92.9 mm, vias 0 -> 1
- net +5VA: track 0.00 -> 87.5 mm
- net Sw2: track 0.00 -> 78.5 mm
- net OUT2: track 0.00 -> 61.5 mm, vias 0 -> 1
- net OUT1: track 0.00 -> 59.2 mm, vias 0 -> 1
- net Net-(Conn5-Pin_2): track 0.00 -> 59.0 mm, vias 0 -> 1
- net IN2: track 0.00 -> 57.3 mm
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- added copper zone on B.Cu, net +3.3V
- removed copper zone on B.Cu, net GND
