File: Scout_Board.kicad_pcb (KiCad board)
At the start: 4 copper layers, 104.1 x 61 mm, 31 parts, among them J1 Conn_01x04_Pin, J10 BBAI_P9, J11 BBAI_P8, J2 Conn_02x07_Odd_Even, J3 705530002, J7 I2C, J8 SPI, Q1 BSS138, Q2 BSS138, Q3 BSS138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

Commit message: Updated board
Parts:
- removed J1: Conn_01x04_Pin, Connector_PinSocket_2.54mm:PinSocket_1x04_P2.54mm_Vertical
- added J5: 5V, Connector_PinSocket_2.54mm:PinSocket_2x05_P2.54mm_Vertical, F.Cu at (267.2, 130.8)
- added J6: GND, Connector_PinSocket_2.54mm:PinSocket_2x05_P2.54mm_Vertical, F.Cu at (257.1, 146.0)
- added J9: Conn_02x04_Counter_Clockwise, Connector_PinSocket_2.54mm:PinSocket_2x04_P2.54mm_Vertical, F.Cu at (171.2, 142.7)
- added JP1: Jumper_2_Open, TestPoint:TestPoint_2Pads_Pitch2.54mm_Drill0.8mm, F.Cu at (258.8, 186.4)
- J10: footprint Connector_PinSocket_2.54mm:PinSocket_2x25_P2.54mm_Vertical -> Custom Library:BBAI-P9; moved to B.Cu
- J11: footprint Connector_PinSocket_2.54mm:PinSocket_2x23_P2.54mm_Vertical -> Custom Library:BBAI-P8; moved to B.Cu
- J7: footprint digikey-footprints:PinHeader_1x2_P2.5mm_Drill1.1mm -> Connector_JST:JST_XH_B2B-XH-AM_1x02_P2.50mm_Vertical
- J8: footprint digikey-footprints:PinHeader_1x4_P2.5mm_Drill1.1mm -> Connector_JST:JST_XH_B4B-XH-AM_1x04_P2.50mm_Vertical
- Q1, Q2, Q3: footprint BSS138:SOT95P240X111-3N -> BSS138W_7_F:SOT-323_DIO
- U2: value ~ -> Steppper motor driver
- moved J7 82.5 mm to (252.7, 136.6), turned to 90 degrees
- moved J10 66.1 mm to (243.8, 137.2)
- moved J11 61.0 mm to (238.8, 185.4)
- moved J8 37.0 mm to (209.3, 145.0), turned to 0 degrees
- moved J3 21.1 mm to (255.2, 153.2)
- moved Conn2 1.80 mm to (179.1, 143.5)
- moved C1 1.78 mm to (246.1, 163.3)
- moved U2 1.51 mm to (247.7, 182.6)
- moved Q1 0.37 mm to (229.3, 165.2), turned to 0 degrees
- moved Q2 0.35 mm to (222.7, 165.2), turned to 0 degrees
- moved Q3 0.08 mm to (216.8, 165.2), turned to 0 degrees
Connections:
- J2 pad 2: unconnected-(J2-Pin_2-Pad2) -> GND
- J3 pad 1: GND -> 5V
- J3 pad 2: 5V -> GND
- J7 pad 1: I2C1_SCL -> I2C1_SDA
- J7 pad 2: I2C1_SDA -> I2C1_SCL
- J8 pad 1: SPI1_CS0 -> SPI1_SCLK
- J8 pad 3: SPI1_SCLK -> SPI1_D0
- J8 pad 4: SPI1_D0 -> SPI1_CS0
- U1 pad J1_12: RxD -> Sys_reset
- U1 pad J1_14: Sys_reset -> RxD
- U1 pad J1_15: Conn1 -> Conn7
- U1 pad J1_16: Conn2 -> Conn5
- U1 pad J1_18: Conn4 -> Conn1
- U1 pad J3_11: unconnected-(U1-GPIO37-PadJ3_11) -> SBC_Power
- U1 pad J3_12: unconnected-(U1-GPIO36-PadJ3_12) -> Wire2
- U1 pad J3_13: unconnected-(U1-GPIO35-PadJ3_13) -> Wire1
- U1 pad J3_15: unconnected-(U1-GPIO45-PadJ3_15) -> Conn8
- U1 pad J3_16: unconnected-(U1-GPIO48-PadJ3_16) -> Conn6
- U1 pad J3_17: unconnected-(U1-GPIO47-PadJ3_17) -> Conn4
- U1 pad J3_18: Wire2 -> Conn2
- U1 pad J3_19: SBC_Power -> unconnected-(U1-USB_D+/GPIO20-PadJ3_19)
- U1 pad J3_20: Wire1 -> unconnected-(U1-USB_D-/GPIO19-PadJ3_20)
Routing:
- net Conn6: track 0.00 -> 42.8 mm
- net Conn8: track 0.00 -> 41.7 mm
- net Conn7: track 0.00 -> 33.5 mm
- net Conn5: track 0.00 -> 32.3 mm
- net Wire1: track 8.67 -> 29.0 mm
- net Conn4: track 26.5 -> 44.0 mm
- net Wire2: track 5.08 -> 22.4 mm
- net SBC_Power: track 5.08 -> 22.4 mm
- net SPI1_CS0: track 36.3 -> 19.5 mm
- net SPI1_D1: track 34.0 -> 17.4 mm
- net Conn1: track 45.9 -> 30.3 mm
- net SPI1_D0: track 34.4 -> 21.8 mm
- net I2C1_SDA: track 26.8 -> 39.0 mm
- net I2C1_SCL: track 29.3 -> 40.8 mm
- net SPI1_SCLK: track 30.8 -> 19.5 mm
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Other:
- board size 104.1 x 61 mm -> 104.1 x 59 mm
- board text added: "1"
- board text added: "10"
- board text added: "11"
- board text added: "12"
- board text added: "2"
- board text added: "35"
- board text added: "45"
- board text added: "46"
- board text added: "47"
- board text added: "48"
- board text added: "9"
- board text added: "DIR"
- board text added: "E1"
- board text added: "E2"
- board text added: "E3"
- board text added: "E4"
- board text added: "EN"
- board text added: "UART"
- board text removed: "23"
