File: lm25116.kicad_sch (KiCad schematic)
At the start: 51 parts, among them U5 LM25116MHX/NOPB, U6 SI7850ADP-T1-GE3, U7 SI7850ADP-T1-GE3

Commit message: New board test
Parts:
- renumbered C4 to C10, C70 to C11, C3 to C12, C11 to C13, C6 to C14, C12 to C15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
