File: Lm25116 power/Lm25116 power.kicad_sch (KiCad schematic)
At the start: 51 parts, among them U1 SI7850ADP-T1-GE3, U2 SI7850ADP-T1-GE3, U3 LM25116MH

Commit message: New board test
Changed lines of the file:
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@@
 	)
 	(junction
+		(at 271.78 88.9)
+		(diameter 0)
+		(color 0 0 0 0)
+	)
+	(junction
 		(at 60.96 66.04)
 		(diameter 0)
@@
 	(wire
 		(pts
+			(xy 271.78 85.09) (xy 271.78 88.9)
+		)
+		(stroke
+			(width 0)
+			(type default)
+		)
+	)
+	(wire
+		(pts
 			(xy 35.56 69.85) (xy 35.56 66.04)
 		)
@@
 	(wire
 		(pts
+			(xy 279.4 86.36) (xy 279.4 88.9)
+		)
+		(stroke
+			(width 0)
+			(type default)
+		)
+	)
+	(wire
+		(pts
 			(xy 19.05 99.06) (xy 19.05 114.3)
 		)
@@
 	(wire
 		(pts
+			(xy 279.4 88.9) (xy 271.78 88.9)
+		)
+		(stroke
+			(width 0)
+			(type default)
+		)
+	)
+	(wire
+		(pts
 			(xy 196.85 49.53) (xy 167.64 49.53)
 		)
@@
 	(symbol
 		(lib_id "power:+5V")
-		(at 271.78 88.9 0)
+		(at 271.78 85.09 0)
 		(unit 1)
 		(exclude_from_sim no)
@@
 		(fields_autoplaced yes)
 		(property "Reference" "#PWR05"
-			(at 271.78 92.71 0)
+			(at 271.78 88.9 0)
 			(effects
 				(font
@@
 		)
 		(property "Value" "+5V"
-			(at 271.78 83.82 0)
+			(at 271.78 80.01 0)
 			(effects
 				(font
@@
 		)
 		(property "Footprint" ""
-			(at 271.78 88.9 0)
+			(at 271.78 85.09 0)
 			(effects
 				(font
@@
 		)
 		(property "Datasheet" ""
-			(at 271.78 88.9 0)
+			(at 271.78 85.09 0)
 			(effects
 				(font
@@
 		)
 		(property "Description" "Power symbol creates a global label with name \"+5V\""
-			(at 271.78 88.9 0)
+			(at 271.78 85.09 0)
 			(effects
 				(font
@@
 					(unit 1)
 				)
+			)
+		)
+	)
+	(symbol
+		(lib_id "power:PWR_FLAG")
+		(at 279.4 86.36 0)
+		(unit 1)
+		(exclude_from_sim no)
+		(in_bom yes)
+		(on_board yes)
+		(dnp no)
+		(fields_autoplaced yes)
+		(property "Reference" "#FLG04"
+			(at 279.4 84.455 0)
+			(effects
+				(font
+					(size 1.27 1.27)
+				)
+				(hide yes)
+			)
+		)
+		(property "Value" "PWR_FLAG"
+			(at 279.4 81.28 0)
+			(effects
+				(font
+					(size 1.27 1.27)
+				)
+			)
+		)
+		(property "Footprint" ""
+			(at 279.4 86.36 0)
+			(effects
+				(font
+					(size 1.27 1.27)
+				)
+				(hide yes)
+			)
+		)
+		(property "Datasheet" "~"
+			(at 279.4 86.36 0)
+			(effects
+				(font
+					(size 1.27 1.27)
+				)
+				(hide yes)
+			)
+		)
+		(property "Description" "Special symbol for telling ERC where power comes from"
+			(at 279.4 86.36 0)
+			(effects
+				(font
+					(size 1.27 1.27)
+				)
+				(hide yes)
+			)
+		)
+		(pin "1"
+		)
+		(instances
+			(project ""
+				(path "/31f273f7-9033-4854-9dd2-6b0faaf8ad00"
+					(reference "#FLG04")
+					(unit 1)
+				)
